Commit message: navigation -intermediate

File: driftbot_ws/src/driftbot_description/urdf/arm_active.xacro (robot description, xacro)
@@ -1,5 +1,5 @@
 <?xml version="1.0"?>
 <robot xmlns:xacro="http://www.ros.org/wiki/xacro">
-  <xacro:property name="arm_scale" value="0.0016 0.0016 0.0016"/>
+  <xacro:property name="arm_scale" value="0.0018 0.0018 0.0018"/>
   <xacro:property name="l1_visual_xyz" value="0 0 -0.0481"/>
   <xacro:property name="l2_visual_xyz" value="0 0 0"/>
@@ -10,7 +10,13 @@
   <xacro:property name="forearm_tip_xyz" value="0 -0.185 0"/>
   <xacro:property name="wrist_tip_xyz" value="0.17751 0 0"/>
-  <xacro:property name="magnet_radius" value="0.08"/>
-  <xacro:property name="magnet_offset_xyz" value="0.09 0 0"/>
-  <!-- AL5D base mounted on torso right side -->
+  <xacro:property name="magnet_gripper_xyz" value="0 0.35 0"/>
+  <!-- magnet R -->
+  <xacro:property name="magnet_radius" value="0.13"/>
+  <xacro:property name="magnet_visual_radius" value="0.13"/>
+  <!-- home rad ref -->
+  <xacro:property name="arm_home_shoulder" value="0.38"/>
+  <xacro:property name="arm_home_elbow" value="-0.88"/>
+  <xacro:property name="arm_home_wrist" value="0.06"/>
+  <!-- arm base -->
   <link name="arm_base_link">
     <visual>
@@ -32,5 +38,5 @@
   <origin xyz="0.0 ${torso_ly/2.0} 0.04" rpy="-1.5708 0 0"/>
 </joint>
-  <!-- Link 1 — shoulder rotation -->
+  <!-- shoulder -->
   <link name="upper_arm_link">
     <visual>
@@ -45,5 +51,5 @@
       <geometry><cylinder radius="0.025" length="0.10"/></geometry>
     </collision>
-    <xacro:inertia_cylinder m="0.187" r="0.025" l="0.10"/>
+    <xacro:inertia_cylinder_z_at m="0.187" r="0.025" l="0.10" ox="0" oy="0" oz="0.05"/>
   </link>
   <joint name="shoulder_joint" type="revolute">
@@ -52,8 +58,9 @@
     <origin xyz="${shoulder_joint_xyz}" rpy="0 3.14159 0"/>
     <axis xyz="0 0 1"/>
-    <limit lower="-1.57" upper="1.57" effort="20.0" velocity="1.0"/>
-    <dynamics damping="0.5" friction="0.2"/>
+    <!-- limit inboard -->
+    <limit lower="-0.18" upper="1.48" effort="20.0" velocity="1.0"/>
+    <dynamics damping="1.2" friction="0.35"/>
   </joint>
-  <!-- Link 2 — elbow -->
+  <!-- elbow -->
   <link name="forearm_link">
     <visual>
@@ -68,5 +75,5 @@
       <geometry><cylinder radius="0.022" length="0.15"/></geometry>
     </collision>
-    <xacro:inertia_cylinder m="0.044" r="0.022" l="0.15"/>
+    <xacro:inertia_cylinder_x_at m="0.044" r="0.022" l="0.15" ox="0.07" oy="0" oz="0"/>
   </link>
   <joint name="elbow_joint" type="revolute">
@@ -75,8 +82,9 @@
     <origin xyz="${elbow_joint_xyz}" rpy="0 1.5708 -1.5708"/>
     <axis xyz="0 0 1"/>
-    <limit lower="-1.57" upper="1.57" effort="15.0" velocity="1.0"/>
-    <dynamics damping="0.4" friction="0.15"/>
+    <!-- no self-hit -->
+    <limit lower="-2.05" upper="0.12" effort="15.0" velocity="1.0"/>
+    <dynamics damping="1.0" friction="0.28"/>
   </joint>
-  <!-- Link 3 — wrist -->
+  <!-- wrist -->
 <link name="wrist_link">
   <visual>
@@ -91,15 +99,15 @@
     <geometry><cylinder radius="0.020" length="0.18"/></geometry>
   </collision>
-  <xacro:inertia_cylinder m="0.207" r="0.020" l="0.18"/>
+  <xacro:inertia_cylinder_x_at m="0.207" r="0.020" l="0.18" ox="0.09" oy="0" oz="0"/>
 </link>
 <joint name="wrist_joint" type="revolute">
   <parent link="forearm_link"/>
   <child  link="wrist_link"/>
-  <origin xyz="${forearm_tip_xyz}" rpy="0 3.14159 1.5708"/>
+  <origin xyz="${forearm_tip_xyz}" rpy="0 3.14159 0"/>
   <axis xyz="0 0 1"/>
-  <limit lower="-1.57" upper="1.57" effort="8.0" velocity="1.5"/>
-  <dynamics damping="0.2" friction="0.1"/>
+  <limit lower="-0.95" upper="1.15" effort="8.0" velocity="1.5"/>
+  <dynamics damping="0.55" friction="0.18"/>
 </joint>
-  <!-- Link 4 — gripper -->
+  <!-- gripper -->
   <link name="gripper_link">
     <visual>
@@ -114,5 +122,5 @@
       <geometry><cylinder radius="0.018" length="0.10"/></geometry>
     </collision>
-    <xacro:inertia_cylinder m="0.081" r="0.018" l="0.10"/>
+    <xacro:inertia_cylinder_x_at m="0.081" r="0.018" l="0.10" ox="0.05" oy="0" oz="0"/>
   </link>
   <joint name="gripper_joint" type="fixed">
@@ -122,4 +130,11 @@
   </joint>
   <link name="magnet_zone_link">
+    <visual>
+      <origin xyz="0 0 0" rpy="0 0 0"/>
+      <geometry>
+        <sphere radius="${magnet_visual_radius}"/>
+      </geometry>
+      <material name="grey"/>
+    </visual>
     <collision name="magnet_zone_collision">
       <origin xyz="0 0 0" rpy="0 0 0"/>
@@ -133,12 +148,12 @@
     <parent link="gripper_link"/>
     <child  link="magnet_zone_link"/>
-    <origin xyz="${magnet_offset_xyz}" rpy="0 0 0"/>
+    <origin xyz="${magnet_gripper_xyz}" rpy="0 0 0"/>
   </joint>
-  <!-- Keep this fixed child link in SDF so DetachableJoint can use it as parent_link. -->
+  <!-- magnet sdf -->
   <gazebo reference="magnet_zone_joint">
     <preserveFixedJoint>true</preserveFixedJoint>
   </gazebo>
   <gazebo reference="magnet_zone_link">
-    <gravity>false</gravity>
+    <turnGravityOff>true</turnGravityOff>
     <sensor name="magnet_zone_contact" type="contact">
       <always_on>true</always_on>
@@ -150,22 +165,17 @@
   </gazebo>
   <gazebo reference="arm_base_link">
-  <material>Gazebo/DarkGrey</material>
-  <gravity>false</gravity>
-</gazebo>
+    <turnGravityOff>true</turnGravityOff>
+  </gazebo>
   <gazebo reference="upper_arm_link">
-  <material>Gazebo/Grey</material>
-  <gravity>false</gravity>
-</gazebo>
+    <turnGravityOff>true</turnGravityOff>
+  </gazebo>
   <gazebo reference="forearm_link">
-  <material>Gazebo/Grey</material>
-  <gravity>false</gravity>
-</gazebo>
+    <turnGravityOff>true</turnGravityOff>
+  </gazebo>
   <gazebo reference="wrist_link">
-  <material>Gazebo/Grey</material>
-  <gravity>false</gravity>
-</gazebo>
+    <turnGravityOff>true</turnGravityOff>
+  </gazebo>
   <gazebo reference="gripper_link">
-  <material>Gazebo/DarkGrey</material>
-  <gravity>false</gravity>
-</gazebo>
+    <turnGravityOff>true</turnGravityOff>
+  </gazebo>
 </robot>

File: driftbot_ws/src/driftbot_description/urdf/arm_cosmetic.xacro (robot description, xacro)
@@ -38,5 +38,5 @@
       <geometry><cylinder radius="0.025" length="0.18"/></geometry>
     </collision>
-    <xacro:inertia_cylinder m="0.30" r="0.025" l="0.18"/>
+    <xacro:inertia_cylinder_z_at m="0.30" r="0.025" l="0.18" ox="0" oy="0" oz="-0.09"/>
   </link>
   <link name="cosm_forearm_link">
@@ -50,5 +50,5 @@
       <geometry><cylinder radius="0.022" length="0.16"/></geometry>
     </collision>
-    <xacro:inertia_cylinder m="0.20" r="0.022" l="0.16"/>
+    <xacro:inertia_cylinder_z_at m="0.20" r="0.022" l="0.16" ox="0" oy="0" oz="-0.08"/>
   </link>
   <link name="cosm_end_link">
@@ -70,18 +70,14 @@
   </joint>
   <gazebo reference="cosm_shoulder_cap_link">
-  <material>Gazebo/DarkGrey</material>
-  <gravity>false</gravity>
-</gazebo>
+    <turnGravityOff>true</turnGravityOff>
+  </gazebo>
   <gazebo reference="cosm_upper_arm_link">
-  <material>Gazebo/Grey</material>
-  <gravity>false</gravity>
-</gazebo>
+    <turnGravityOff>true</turnGravityOff>
+  </gazebo>
   <gazebo reference="cosm_forearm_link">
-  <material>Gazebo/Grey</material>
-  <gravity>false</gravity>
-</gazebo>
+    <turnGravityOff>true</turnGravityOff>
+  </gazebo>
   <gazebo reference="cosm_end_link">
-  <material>Gazebo/DarkGrey</material>
-  <gravity>false</gravity>
-</gazebo>
+    <turnGravityOff>true</turnGravityOff>
+  </gazebo>
 </robot>

File: driftbot_ws/src/driftbot_description/urdf/base.xacro (robot description, xacro)
@@ -9,5 +9,5 @@
   <xacro:property name="wheel_width"  value="0.10"/>
   <xacro:property name="wheel_mass"   value="0.5"/>
-  <!-- Lateral offset of wheel joint from base_link (half track width). Was 0.235; increased so tires sit outside the chassis box (base_len_y/2 = 0.21). -->
+  <!-- half track -->
   <xacro:property name="wheel_track_half_y" value="0.275"/>
   <link name="base_footprint"/>
@@ -32,5 +32,4 @@
   </link>
   <gazebo reference="base_link">
-    <material>Gazebo/DarkGrey</material>
     <mu1>0.8</mu1>
     <mu2>0.8</mu2>
@@ -50,7 +49,4 @@
     <xacro:inertia_box m="1.324" lx="0.732" ly="0.488" lz="0.244"/>
   </link>
-  <gazebo reference="top_shell_link">
-    <material>Gazebo/DarkGrey</material>
-  </gazebo>
   <joint name="base_top_joint" type="fixed">
     <parent link="base_link"/>
@@ -73,5 +69,5 @@
         </geometry>
       </collision>
-      <xacro:inertia_cylinder m="${wheel_mass}" r="${wheel_radius}" l="${wheel_width}"/>
+      <xacro:inertia_cylinder_y_at m="${wheel_mass}" r="${wheel_radius}" l="${wheel_width}" ox="0" oy="0" oz="0"/>
     </link>
     <joint name="wheel_${name}_joint" type="continuous">
@@ -83,5 +79,4 @@
     </joint>
     <gazebo reference="wheel_${name}">
-      <material>Gazebo/Black</material>
       <mu1>1.2</mu1>
       <mu2>1.2</mu2>

File: driftbot_ws/src/driftbot_description/urdf/inertia_macros.xacro (robot description, xacro)
@@ -12,6 +12,8 @@
     </inertial>
   </xacro:macro>
-  <xacro:macro name="inertia_cylinder" params="m r l">
+  <!-- cyl +Z -->
+  <xacro:macro name="inertia_cylinder_z_at" params="m r l ox oy oz">
     <inertial>
+      <origin xyz="${ox} ${oy} ${oz}" rpy="0 0 0"/>
       <mass value="${m}"/>
       <inertia
@@ -22,4 +24,33 @@
         izz="${0.5*m*r*r}"/>
     </inertial>
+  </xacro:macro>
+  <!-- cyl +X -->
+  <xacro:macro name="inertia_cylinder_x_at" params="m r l ox oy oz">
+    <inertial>
+      <origin xyz="${ox} ${oy} ${oz}" rpy="0 0 0"/>
+      <mass value="${m}"/>
+      <inertia
+        ixx="${0.5*m*r*r}"
+        ixy="0" ixz="0"
+        iyy="${(1.0/12.0)*m*(3*r*r + l*l)}"
+        iyz="0"
+        izz="${(1.0/12.0)*m*(3*r*r + l*l)}"/>
+    </inertial>
+  </xacro:macro>
+  <!-- cyl +Y -->
+  <xacro:macro name="inertia_cylinder_y_at" params="m r l ox oy oz">
+    <inertial>
+      <origin xyz="${ox} ${oy} ${oz}" rpy="0 0 0"/>
+      <mass value="${m}"/>
+      <inertia
+        ixx="${(1.0/12.0)*m*(3*r*r + l*l)}"
+        ixy="0" ixz="0"
+        iyy="${0.5*m*r*r}"
+        iyz="0"
+        izz="${(1.0/12.0)*m*(3*r*r + l*l)}"/>
+    </inertial>
+  </xacro:macro>
+  <xacro:macro name="inertia_cylinder" params="m r l">
+    <xacro:inertia_cylinder_z_at m="${m}" r="${r}" l="${l}" ox="0" oy="0" oz="0"/>
   </xacro:macro>
   <xacro:macro name="inertia_sphere" params="m r">

File: driftbot_ws/src/driftbot_description/urdf/robot.urdf.xacro (robot description, xacro)
@@ -16,7 +16,7 @@
       <right_joint>wheel_fr_joint</right_joint>
       <right_joint>wheel_rr_joint</right_joint>
-      <!-- Track width: 2 * wheel_track_half_y (base.xacro). -->
+      <!-- track width -->
       <wheel_separation>0.55</wheel_separation>
-      <wheel_radius>0.10</wheel_radius>
+      <wheel_radius>0.165</wheel_radius>
       <max_linear_velocity>0.8</max_linear_velocity>
       <max_angular_velocity>1.5</max_angular_velocity>
@@ -26,4 +26,5 @@
       <topic>cmd_vel</topic>
       <odom_topic>odom</odom_topic>
+      <!-- no gz /tf -->
       <tf_topic>tf</tf_topic>
       <frame_id>odom</frame_id>
@@ -37,28 +38,49 @@
     </plugin>
   </gazebo>
+  <!-- arm topics -->
   <gazebo>
-    <plugin filename="gz-sim-sensors-system"
-            name="gz::sim::systems::Sensors">
-      <render_engine>ogre2</render_engine>
+    <plugin filename="gz-sim-joint-position-controller-system"
+            name="gz::sim::systems::JointPositionController">
+      <joint_name>shoulder_joint</joint_name>
+      <topic>arm_cmd_shoulder</topic>
+      <p_gain>50</p_gain>
+      <i_gain>0.02</i_gain>
+      <d_gain>0.35</d_gain>
+      <cmd_max>80</cmd_max>
+      <cmd_min>-80</cmd_min>
     </plugin>
   </gazebo>
-  <!-- Contact system is required by TouchPlugin and contact sensors. -->
+  <gazebo>
+    <plugin filename="gz-sim-joint-position-controller-system"
+            name="gz::sim::systems::JointPositionController">
+      <joint_name>elbow_joint</joint_name>
+      <topic>arm_cmd_elbow</topic>
+      <p_gain>50</p_gain>
+      <i_gain>0.02</i_gain>
+      <d_gain>0.35</d_gain>
+      <cmd_max>80</cmd_max>
+      <cmd_min>-80</cmd_min>
+    </plugin>
+  </gazebo>
+  <gazebo>
+    <plugin filename="gz-sim-joint-position-controller-system"
+            name="gz::sim::systems::JointPositionController">
+      <joint_name>wrist_joint</joint_name>
+      <topic>arm_cmd_wrist</topic>
+      <p_gain>40</p_gain>
+      <i_gain>0.02</i_gain>
+      <d_gain>0.25</d_gain>
+      <cmd_max>60</cmd_max>
+      <cmd_min>-60</cmd_min>
+    </plugin>
+  </gazebo>
+  <!-- lidar world plugin -->
+  <!-- contacts -->
   <gazebo>
     <plugin filename="gz-sim-contact-system"
-            name="gz::sim::systems::Contact"/>
+            name="gz::sim::systems::Contact">
+    </plugin>
   </gazebo>
-  <!-- Magnetic pickup behavior for floor objects.
-       Targets in home.sdf:
-         - can
-         - ball
-         - toy_block_1
-         - toy_block_2
-         - toy_cylinder_1
-         - toy_block_3
-       All targets use child_link=link.
-       Control topics (Gazebo transport):
-         - /magnet_on  (gz.msgs.Empty): attach targets
-         - /magnet_off (gz.msgs.Empty): detach targets
-  -->
+  <!-- pick attach -->
   <gazebo>
     <plugin filename="gz-sim-detachable-joint-system"
@@ -118,34 +140,4 @@
     <plugin filename="gz-sim-triggered-publisher-system"
             name="gz::sim::systems::TriggeredPublisher">
-      <input type="gz.msgs.Empty" topic="/magnet_on"/>
-      <output type="gz.msgs.Empty" topic="/can/attach"/>
-    </plugin>
-    <plugin filename="gz-sim-triggered-publisher-system"
-            name="gz::sim::systems::TriggeredPublisher">
-      <input type="gz.msgs.Empty" topic="/magnet_on"/>
-      <output type="gz.msgs.Empty" topic="/ball/attach"/>
-    </plugin>
-    <plugin filename="gz-sim-triggered-publisher-system"
-            name="gz::sim::systems::TriggeredPublisher">
-      <input type="gz.msgs.Empty" topic="/magnet_on"/>
-      <output type="gz.msgs.Empty" topic="/toy_block_1/attach"/>
-    </plugin>
-    <plugin filename="gz-sim-triggered-publisher-system"
-            name="gz::sim::systems::TriggeredPublisher">
-      <input type="gz.msgs.Empty" topic="/magnet_on"/>
-      <output type="gz.msgs.Empty" topic="/toy_block_2/attach"/>
-    </plugin>
-    <plugin filename="gz-sim-triggered-publisher-system"
-            name="gz::sim::systems::TriggeredPublisher">
-      <input type="gz.msgs.Empty" topic="/magnet_on"/>
-      <output type="gz.msgs.Empty" topic="/toy_cylinder_1/attach"/>
-    </plugin>
-    <plugin filename="gz-sim-triggered-publisher-system"
-            name="gz::sim::systems::TriggeredPublisher">
-      <input type="gz.msgs.Empty" topic="/magnet_on"/>
-      <output type="gz.msgs.Empty" topic="/toy_block_3/attach"/>
-    </plugin>
-    <plugin filename="gz-sim-triggered-publisher-system"
-            name="gz::sim::systems::TriggeredPublisher">
       <input type="gz.msgs.Empty" topic="/magnet_off"/>
       <output type="gz.msgs.Empty" topic="/can/detach"/>

File: driftbot_ws/src/driftbot_description/urdf/ros2_control.xacro (robot description, xacro)
@@ -1,40 +1,4 @@
 <?xml version="1.0"?>
 <robot xmlns:xacro="http://www.ros.org/wiki/xacro">
-  <ros2_control name="driftbot_arm" type="system">
-    <hardware>
-      <plugin>gz_ros2_control/GazeboSimSystem</plugin>
-    </hardware>
-    <joint name="shoulder_joint">
-      <command_interface name="position">
-        <param name="min">-1.57</param>
-        <param name="max"> 1.57</param>
-      </command_interface>
-      <state_interface name="position"/>
-      <state_interface name="velocity"/>
-    </joint>
-    <joint name="elbow_joint">
-      <command_interface name="position">
-        <param name="min">-2.35</param>
-        <param name="max"> 0.10</param>
-      </command_interface>
-      <state_interface name="position"/>
-      <state_interface name="velocity"/>
-    </joint>
-    <joint name="wrist_joint">
-      <command_interface name="position">
-        <param name="min">-1.57</param>
-        <param name="max"> 1.57</param>
-      </command_interface>
-      <state_interface name="position"/>
-      <state_interface name="velocity"/>
-    </joint>
-  </ros2_control>
-  <!-- TODO: uncomment after driftbot_bringup is built
-  <gazebo>
-    <plugin filename="gz_ros2_control-system"
-            name="gz_ros2_control::GazeboSimROS2ControlPlugin">
-      <parameters>$(find driftbot_bringup)/config/ros2_control.yaml</parameters>
-    </plugin>
-  </gazebo>
-  -->
+  <!-- passive arm -->
 </robot>

File: driftbot_ws/src/driftbot_description/urdf/sensors.xacro (robot description, xacro)
@@ -11,5 +11,5 @@
     <geometry><cylinder radius="0.020" length="0.040"/></geometry>
   </collision>
-  <xacro:inertia_cylinder m="0.08" r="0.020" l="0.040"/>
+  <xacro:inertia_cylinder_y_at m="0.08" r="0.020" l="0.040" ox="0" oy="0" oz="0"/>
 </link>
   <link name="camera_optical_link"/>
@@ -17,5 +17,5 @@
     <parent link="torso_link"/>
     <child  link="camera_link"/>
-    <origin xyz="0.095 0.0 0.08" rpy="0 0 0"/>
+    <origin xyz="0.095 0.0 -0.08" rpy="0 0 0"/>
   </joint>
   <joint name="camera_optical_joint" type="fixed">
@@ -25,5 +25,4 @@
   </joint>
   <gazebo reference="camera_link">
-    <material>Gazebo/Black</material>
     <sensor name="driftbot_camera" type="camera">
       <always_on>true</always_on>
@@ -32,4 +31,6 @@
       <topic>/camera/image_raw</topic>
       <camera>
+        <!-- ogre mask -->
+        <visibility_mask>268435455</visibility_mask>
         <horizontal_fov>1.047</horizontal_fov>
         <image>
@@ -62,6 +63,6 @@
   <origin xyz="0.239 0.0 0.24" rpy="0 0 0"/>
 </joint>
+  <!-- 2d scan -->
   <gazebo reference="lidar_link">
-    <material>Gazebo/Black</material>
     <sensor name="driftbot_lidar" type="gpu_lidar">
       <always_on>true</always_on>
@@ -70,4 +71,5 @@
       <topic>/scan</topic>
       <lidar>
+        <visibility_mask>268435455</visibility_mask>
         <scan>
           <horizontal>
@@ -83,9 +85,4 @@
           <resolution>0.01</resolution>
         </range>
-        <noise>
-          <type>gaussian</type>
-          <mean>0.0</mean>
-          <stddev>0.005</stddev>
-        </noise>
       </lidar>
     </sensor>

File: driftbot_ws/src/driftbot_description/urdf/torso.xacro (robot description, xacro)
@@ -31,5 +31,5 @@
       <origin xyz="0 0 0" rpy="0 0 0"/>
       <geometry><box size="${face_lx} ${face_ly} ${face_lz}"/></geometry>
-      <material name="cyan"/>
+      <material name="grey"/>
     </visual>
     <collision>
@@ -44,5 +44,5 @@
   <origin xyz="${torso_lx/2.0 + face_lx/2.0} 0.0 0.24" rpy="0 0 0"/>
 </joint>
-<!-- "<"> glyph -->
+<!-- xml escape -->
 <link name="glyph_lt_top_link">
   <visual>
@@ -51,4 +51,8 @@
     <material name="burgundy"/>
   </visual>
+  <collision>
+    <origin xyz="0 0 0" rpy="0 0 0"/>
+    <geometry><box size="0.003 0.032 0.006"/></geometry>
+  </collision>
   <xacro:inertia_box m="0.0015" lx="0.003" ly="0.032" lz="0.006"/>
 </link>
@@ -64,4 +68,8 @@
     <material name="burgundy"/>
   </visual>
+  <collision>
+    <origin xyz="0 0 0" rpy="0 0 0"/>
+    <geometry><box size="0.003 0.032 0.006"/></geometry>
+  </collision>
   <xacro:inertia_box m="0.0015" lx="0.003" ly="0.032" lz="0.006"/>
 </link>
@@ -77,4 +85,8 @@
     <material name="burgundy"/>
   </visual>
+  <collision>
+    <origin xyz="0 0 0" rpy="0 0 0"/>
+    <geometry><box size="0.003 0.008 0.028"/></geometry>
+  </collision>
   <xacro:inertia_box m="0.0015" lx="0.003" ly="0.008" lz="0.028"/>
 </link>
@@ -90,4 +102,8 @@
     <material name="burgundy"/>
   </visual>
+  <collision>
+    <origin xyz="0 0 0" rpy="0 0 0"/>
+    <geometry><box size="0.003 0.008 0.028"/></geometry>
+  </collision>
   <xacro:inertia_box m="0.0015" lx="0.003" ly="0.008" lz="0.028"/>
 </link>
@@ -103,4 +119,8 @@
     <material name="burgundy"/>
   </visual>
+  <collision>
+    <origin xyz="0 0 0" rpy="0 0 0"/>
+    <geometry><box size="0.003 0.032 0.006"/></geometry>
+  </collision>
   <xacro:inertia_box m="0.0015" lx="0.003" ly="0.032" lz="0.006"/>
 </link>
@@ -116,4 +136,8 @@
       <material name="burgundy"/>
   </visual>
+  <collision>
+    <origin xyz="0 0 0" rpy="0 0 0"/>
+    <geometry><box size="0.003 0.032 0.006"/></geometry>
+  </collision>
   <xacro:inertia_box m="0.0015" lx="0.003" ly="0.032" lz="0.006"/>
 </link>
@@ -123,11 +147,3 @@
   <origin xyz="0.010 -0.060 -0.016" rpy="-0.95 0 0"/>
 </joint>
-  <gazebo reference="torso_link"/>
-<gazebo reference="face_panel_link"><material>Gazebo/Grey</material></gazebo>
-<gazebo reference="glyph_lt_top_link"/>
-<gazebo reference="glyph_lt_bottom_link"/>
-<gazebo reference="glyph_quote_left_link"/>
-<gazebo reference="glyph_quote_right_link"/>
-<gazebo reference="glyph_gt_top_link"/>
-<gazebo reference="glyph_gt_bottom_link"/>
 </robot>

Commit message: prelim -navigation. not final(experimental)

File: driftbot_ws/src/driftbot_description/urdf/arm_active.xacro (robot description, xacro)
@@ -1,5 +1,5 @@
 <?xml version="1.0"?>
 <robot xmlns:xacro="http://www.ros.org/wiki/xacro">
-  <xacro:property name="arm_scale" value="0.0018 0.0018 0.0018"/>
+  <xacro:property name="arm_scale" value="0.0016 0.0016 0.0016"/>
   <xacro:property name="l1_visual_xyz" value="0 0 -0.0481"/>
   <xacro:property name="l2_visual_xyz" value="0 0 0"/>
@@ -58,6 +58,6 @@
     <origin xyz="${shoulder_joint_xyz}" rpy="0 3.14159 0"/>
     <axis xyz="0 0 1"/>
-    <!-- limit inboard -->
-    <limit lower="-0.18" upper="1.48" effort="20.0" velocity="1.0"/>
+    <!-- limit inboard; lower ≤ stage3 shoulder (e.g. -0.30); small margin for controller -->
+    <limit lower="-0.66" upper="1.48" effort="20.0" velocity="1.0"/>
     <dynamics damping="1.2" friction="0.35"/>
   </joint>
@@ -106,5 +106,5 @@
   <origin xyz="${forearm_tip_xyz}" rpy="0 3.14159 0"/>
   <axis xyz="0 0 1"/>
-  <limit lower="-0.95" upper="1.15" effort="8.0" velocity="1.5"/>
+  <limit lower="-1.38" upper="1.15" effort="8.0" velocity="1.5"/>
   <dynamics damping="0.55" friction="0.18"/>
 </joint>

File: driftbot_ws/src/driftbot_description/urdf/sensors.xacro (robot description, xacro)
@@ -88,3 +88,24 @@
     </sensor>
   </gazebo>
+  <!-- World-frame yaw for in-place turns (avoids diff-drive odom yaw integration error). -->
+  <gazebo reference="base_link">
+    <sensor name="base_imu" type="imu">
+      <always_on>true</always_on>
+      <update_rate>100</update_rate>
+      <visualize>false</visualize>
+      <topic>imu</topic>
+      <imu>
+        <angular_velocity>
+          <x><noise type="gaussian"><mean>0</mean><stddev>1e-4</stddev></noise></x>
+          <y><noise type="gaussian"><mean>0</mean><stddev>1e-4</stddev></noise></y>
+          <z><noise type="gaussian"><mean>0</mean><stddev>1e-4</stddev></noise></z>
+        </angular_velocity>
+        <linear_acceleration>
+          <x><noise type="gaussian"><mean>0</mean><stddev>0.01</stddev></noise></x>
+          <y><noise type="gaussian"><mean>0</mean><stddev>0.01</stddev></noise></y>
+          <z><noise type="gaussian"><mean>0</mean><stddev>0.01</stddev></noise></z>
+        </linear_acceleration>
+      </imu>
+    </sensor>
+  </gazebo>
 </robot>
